File: reverse_ecobeemux_175-00011-revD.kicad_sch (KiCad schematic)
At the start: 24 parts, among them J1 Conn_01x04, J2 Conn_01x05, U1 MOC3063M, U2 MOC3063M

Commit message: Reverse complete. Added board shots.
Parts:
- removed V1, V2: Varistor_US, symbol Device:Varistor_US
- added V1, V2: >60V, symbol Device:D_TVS
- C2, C4: value C -> 3.3n
Connections:
- net FAN: now also V1.1 (A1)
- net HEAT: now also V2.2 (A2)
- net at C4.1, DQ2.2 (A2), R4.2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: now also V2.1 (A1)
- net at C2.2, DQ1.2 (A2), R2.2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: now also V1.2 (A2)
- net 24VAC_N renamed GND
Other:
- note added: "C2/C4 values are guesses/approximations. V1/V2 components are unlabeled and are guesses. They may be MOVs, varistors, etc. They do not conduct at any voltage up to 60V."
- note added: "COOL signal is not multiplexed, it is simply conducted from pin 4 to pin 5 out."
- note added: "GND is AC neutral"
- note added: "Home HVAC signaling is 24VAC_{rms} (unregulated) ladder logic. On PEK line, a positive half-wave rectified AC signal of sufficient magnitude turns on U1 which will supply AC from J2 pin 1 to J2 pin 3 at next zero crossing. A negative half-wave rectified signal will do the same at J2 pin 4 from J2 pin 1. Applying a full AC signal will turn both on at the same time."
- note added: "J1 is push-in spring contact wire connector with 4 pins. J2 is 5-wire pigtail wires."
- note added: "J1 pin hole labels"
- note added: "J2 wire sleeve+board labels and sleeve colors"
- note added: "R/red C/blue G/green W/grey Y/yellow"
- note added: "Representative doorbell transformer checked is about 19.2V_{rms} or 54V pk-to-pk."
- note added: "Turn on current (I_{FT}) of U1 emitter is 5mA. At 6mA: pin 2 of U1 is at 0V (ref) pin 1 of U1 is at 1.5V (max MOC3063M spec) drop across R8 is 900mV (IR) cathode of D3 is at 2.40V (sum) drop across R8 is 14.94V (IR) cathode of D1 is at 17.34V (sum) drop across D1 is 855mV (spec max at 10mA) anode of D1 is at 18.89V (sum) So PEK must go to at least 18.89V peak to turn on U1 and FAN. Ripple at 6mA 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"
- note added: "With capacitor drain at non-peak voltages and ripple due to half-wave rectification about 22V peak needed on PEK at 60 Hz to turn on output signal full duty cycle (5mA at MOC emitter). As PEK is likely derived from the AC source with a diode 22.7V peak would be needed on AC source before recification."
- note added: "pin 1 has dot on board"
- note removed: "R C Gn W Y"
- note removed: "Representative doorbell transformer I checked is about 19.2V_{rms} or 54V pk-to-pk."
- note removed: "Turn on current (I_{FT}) of U1 emitter is 5mA. At 5mA: pin 2 of U1 is at 0V (ref) pin 1 of U1 is at 1.3V (MOC3063M spec) drop across R8 is 750mV (IR) cathode of D3 is at 2.05V (sum) drop across R8 is 14.7V (IR) cathode of D1 is at 16.75V (sum) drop across D1 is 0.7V (spec) anode of D1 is at 17.45V (sum) So PEK must go to at least 17.5V to turn on U1 and FAN."
- title: (none) -> EcoBee power extender kit 175-00011 rev D
- moved on the sheet: C1, C2, C4, C6, D1, D2, D3, D4, DQ1, DQ2, J1, J2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

Commit message: Added README.md including pictures. Added pdf version of schematic. Made some revisions.
Parts:
- renumbered DQ1 to Q1, DQ2 to Q2
Other:
- note added: "R G Y W"
- note removed: "R Gn Y W"
Changed lines of the file:
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@@
 		)
 	)
-	(text "R\nGn\nY\nW"
+	(text "R\nG\nY\nW"
 		(exclude_from_sim no)
 		(at 85.598 81.534 0)
@@
 	)
 	(junction
-		(at 132.08 97.79)
-		(diameter 0)
-		(color 0 0 0 0)
-	)
-	(junction
 		(at 133.35 97.79)
 		(diameter 0)
@@
 	)
 	(junction
+		(at 162.56 97.79)
+		(diameter 0)
+		(color 0 0 0 0)
+	)
+	(junction
 		(at 146.05 82.55)
 		(diameter 0)
@@
 	(wire
 		(pts
+			(xy 133.35 97.79) (xy 132.08 97.79)
+		)
+		(stroke
+			(width 0)
+			(type default)
+		)
+	)
+	(wire
+		(pts
 			(xy 162.56 124.46) (xy 172.72 124.46)
 		)
@@
 	(wire
 		(pts
+			(xy 146.05 97.79) (xy 133.35 97.79)
+		)
+		(stroke
+			(width 0)
+			(type default)
+		)
+	)
+	(wire
+		(pts
 			(xy 199.39 124.46) (xy 205.74 124.46)
 		)
@@
 	(wire
 		(pts
-			(xy 123.19 97.79) (xy 132.08 97.79)
+			(xy 162.56 97.79) (xy 147.32 97.79)
 		)
 		(stroke
@@
 	(wire
 		(pts
-			(xy 121.92 82.55) (xy 118.11 82.55)
+			(xy 162.56 97.79) (xy 168.91 97.79)
 		)
 		(stroke
@@
 	(wire
 		(pts
-			(xy 147.32 97.79) (xy 168.91 97.79)
+			(xy 121.92 82.55) (xy 118.11 82.55)
 		)
 		(stroke
@@
 	(wire
 		(pts
-			(xy 133.35 97.79) (xy 146.05 97.79)
-		)
-		(stroke
-			(width 0)
-			(type default)
-		)
-	)
-	(wire
-		(pts
 			(xy 147.32 113.03) (xy 147.32 109.22)
 		)
@@
 	(wire
 		(pts
-			(xy 132.08 97.79) (xy 133.35 97.79)
-		)
-		(stroke
-			(width 0)
-			(type default)
-		)
-	)
-	(wire
-		(pts
 			(xy 132.08 97.79) (xy 132.08 93.98)
 		)
@@
 	(wire
 		(pts
-			(xy 123.19 97.79) (xy 123.19 99.06)
+			(xy 162.56 97.79) (xy 162.56 100.33)
 		)
 		(stroke
@@
 		(dnp no)
 		(fields_autoplaced yes)
-		(property "Reference" "DQ1"
+		(property "Reference" "Q1"
 			(at 209.55 75.5014 0)
 			(effects
@@
 			)
 		)
-		(property "Datasheet" "~"
+		(property "Datasheet" "https://www.jjm.com/pdf/kkg/ACJT410-10K.pdf"
 			(at 205.74 76.2 90)
 			(effects
@@
 			(project ""
 				(path "/e587ab55-cee7-4136-afa9-28e1a9e31271"
-					(reference "DQ1")
+					(reference "Q1")
 					(unit 1)
 				)
@@
 		(on_board yes)
 		(dnp no)
-		(property "Reference" "DQ2"
+		(property "Reference" "Q2"
 			(at 209.55 116.2684 0)
 			(effects
@@
 			)
 		)
-		(property "Datasheet" "~"
+		(property "Datasheet" "https://www.jjm.com/pdf/kkg/ACJT410-10K.pdf"
 			(at 205.74 118.11 90)
 			(effects
@@
 			(project "reverse_ecobeemux_175-00011-revD"
 				(path "/e587ab55-cee7-4136-afa9-28e1a9e31271"
-					(reference "DQ2")
+					(reference "Q2")
 					(unit 1)
 				)
@@
 	(symbol
 		(lib_id "power:GND")
-		(at 123.19 99.06 0)
+		(at 162.56 100.33 0)
 		(unit 1)
 		(exclude_from_sim no)
@@
 		(fields_autoplaced yes)
 		(property "Reference" "#PWR04"
-			(at 123.19 105.41 0)
+			(at 162.56 106.68 0)
 			(effects
 				(font
@@
 		)
 		(property "Value" "GND"
-			(at 123.19 104.14 0)
+			(at 162.56 105.41 0)
 			(effects
 				(font
@@
 		)
 		(property "Footprint" ""
-			(at 123.19 99.06 0)
+			(at 162.56 100.33 0)
 			(effects
 				(font
@@
 		)
 		(property "Datasheet" ""
-			(at 123.19 99.06 0)
+			(at 162.56 100.33 0)
 			(effects
 				(font
@@
 		)
 		(property "Description" "Power symbol creates a global label with name \"GND\" , ground"
-			(at 123.19 99.06 0)
+			(at 162.56 100.33 0)
 			(effects
 				(font

Commit message: Added footprints to many devices.
Parts:
- C1, C6: footprint (none) -> Capacitor_SMD:CP_Elec_8x5.4
- C2, C4: footprint (none) -> Capacitor_SMD:C_0402_1005Metric
- Q1, Q2: footprint (none) -> Package_TO_SOT_SMD:TO-252-2
- R10, R8: footprint (none) -> Resistor_SMD:R_0402_1005Metric
- R2, R3, R4, R5: footprint (none) -> Resistor_SMD:R_0805_2012Metric
- R7, R9: footprint (none) -> Resistor_SMD:R_1206_3216Metric
- U1, U2: footprint (none) -> Package_DIP:SMDIP-6_W9.53mm
- V1, V2: footprint (none) -> Diode_SMD:D_0603_1608Metric
Other:
- note added: "All diodes are SOT-23 with cathode at pin 3 and anode at pin 1."
Changed lines of the file:
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@@
 		)
 	)
+	(text "All diodes are SOT-23 with cathode at pin 3\nand anode at pin 1."
+		(exclude_from_sim no)
+		(at 138.684 66.294 0)
+		(effects
+			(font
+				(size 1.27 1.27)
+			)
+		)
+	)
 	(text "R\nG\nY\nW"
 		(exclude_from_sim no)
@@
 			)
 		)
-		(property "Footprint" ""
+		(property "Footprint" "Capacitor_SMD:C_0402_1005Metric"
 			(at 218.7448 111.76 0)
 			(effects
@@
 			)
 		)
-		(property "Footprint" ""
+		(property "Footprint" "Diode_SMD:D_0603_1608Metric"
 			(at 229.87 115.57 0)
 			(effects
@@
 			)
 		)
-		(property "Footprint" ""
+		(property "Footprint" "Package_TO_SOT_SMD:TO-252-2"
 			(at 207.645 75.565 90)
 			(effects
@@
 			)
 		)
-		(property "Footprint" ""
+		(property "Footprint" "Resistor_SMD:R_0402_1005Metric"
 			(at 154.686 112.014 90)
 			(effects
@@
 			)
 		)
-		(property "Footprint" ""
+		(property "Footprint" "Resistor_SMD:R_0805_2012Metric"
 			(at 197.104 68.834 90)
 			(effects
@@
 			)
 		)
-		(property "Footprint" ""
+		(property "Footprint" "Resistor_SMD:R_0402_1005Metric"
 			(at 153.416 81.534 90)
 			(effects
@@
 			)
 		)
-		(property "Footprint" ""
+		(property "Footprint" "Resistor_SMD:R_1206_3216Metric"
 			(at 138.176 81.534 90)
 			(effects
@@
 			)
 		)
-		(property "Footprint" ""
+		(property "Footprint" "Package_TO_SOT_SMD:TO-252-2"
 			(at 207.645 118.745 90)
 			(effects
@@
 			)
 		)
-		(property "Footprint" ""
+		(property "Footprint" "Package_DIP:SMDIP-6_W9.53mm"
 			(at 175.26 77.47 0)
 			(effects
@@
 			)
 		)
-		(property "Footprint" ""
+		(property "Footprint" "Resistor_SMD:R_1206_3216Metric"
 			(at 139.446 112.014 90)
 			(effects
@@
 			)
 		)
-		(property "Footprint" ""
+		(property "Footprint" "Resistor_SMD:R_0805_2012Metric"
 			(at 195.834 123.444 90)
 			(effects
@@
 			)
 		)
-		(property "Footprint" ""
+		(property "Footprint" "Capacitor_SMD:C_0402_1005Metric"
 			(at 218.7448 76.2 0)
 			(effects
@@
 			)
 		)
-		(property "Footprint" ""
+		(property "Footprint" "Package_DIP:SMDIP-6_W9.53mm"
 			(at 175.26 127 0)
 			(effects
@@
 			)
 		)
-		(property "Footprint" ""
+		(property "Footprint" "Diode_SMD:D_0603_1608Metric"
 			(at 229.87 80.01 0)
 			(effects
@@
 			)
 		)
-		(property "Footprint" ""
+		(property "Footprint" "Capacitor_SMD:CP_Elec_8x5.4"
 			(at 132.08 90.17 0)
 			(effects
@@
 			)
 		)
-		(property "Footprint" ""
+		(property "Footprint" "Capacitor_SMD:CP_Elec_8x5.4"
 			(at 133.35 105.41 0)
 			(effects
@@
 			)
 		)
-		(property "Footprint" ""
+		(property "Footprint" "Resistor_SMD:R_0805_2012Metric"
 			(at 242.824 123.444 90)
 			(effects
@@
 			)
 		)
-		(property "Footprint" ""
+		(property "Footprint" "Resistor_SMD:R_0805_2012Metric"
 			(at 242.824 68.834 90)
 			(effects
